Commit message: Fix name

File: v2mini_gazebo/urdf/transmission/v2mini_head.transmission.xacro (robot description, xacro)
@@ -1,5 +1,5 @@
 <?xml version="1.0"?>
 <robot xmlns:xacro="http://ros.org/wiki/xacro">
-  <xacro:macro name="v2mini_arm_transmission" params="prefix">
+  <xacro:macro name="v2mini_head_transmission" params="prefix">
    <transmission name="${prefix}neck_tilt">
       <type>transmission_interface/SimpleTransmission</type>
