Commit message: Fix name

File: v2mini_gazebo/urdf/transmission/v2mini_torso.transmission.xacro (robot description, xacro)
@@ -4,5 +4,5 @@
    <transmission name="${prefix}torso_slide_trans">
       <type>transmission_interface/SimpleTransmission</type>
-      <joint name="${prefix}arm_joint1">
+      <joint name="${prefix}torso_slide">
         <hardwareInterface>PositionJointInterface</hardwareInterface>
       </joint>
