Commit message: Added controllers to gazebo

File: v2mini_description/urdf/v2mini_robot.urdf.xacro (robot description, xacro)
@@ -28,4 +28,20 @@
   <!-- r200 sensor -->
   <include filename="$(find v2mini_description)/urdf/sensors/r200.urdf.xacro" />
+ <!-- join the body with head -->
+  <joint name="neckpan" type="revolute">
+    <parent link="torso_link"/>
+    <child link="neck_link"/>
+    <axis xyz="0 0 1"/>
+    <origin xyz="0 0 0"/>
+    <limit effort="10" lower="-2.9" upper="2.9" velocity="10"/>
+  </joint>
+  <!-- join the body with arm -->
+  <joint name="shoulder" type="fixed">
+    <parent link="torso_link"/>
+    <child link="arm_link1"/>
+    <origin xyz="0 0 0"/>
+  </joint>
   <xacro:body/>
+  <xacro:head/>
+  <xacro:arm/>
 </robot>

File: v2mini_gazebo/urdf/v2mini_robot.gazebo.xacro (robot description, xacro)
@@ -13,4 +13,14 @@
     </plugin>
   </gazebo>
+  <!-- Planar move base plugin -->
+   <gazebo>
+    <plugin name="object_controller" filename="libgazebo_ros_planar_move.so">
+      <commandTopic>cmd_vel</commandTopic>
+      <odometryTopic>odom</odometryTopic>
+      <odometryFrame>odom</odometryFrame>
+      <odometryRate>20.0</odometryRate>
+      <robotBaseFrame>base_footprint</robotBaseFrame>
+    </plugin>
+ </gazebo>
   <gazebo>
     <plugin name="gazebo_imu" filename="libgazebo_ros_imu.so">
