Commit message: Added base footprint

File: v2mini_description/urdf/v2mini_body.urdf.xacro (robot description, xacro)
@@ -35,4 +35,5 @@
     </collision>
   </link>
+  <link name="base_footprint"/>
   <xacro:wheel prefix="front" reflect="-1" rotate="0" front_set="1"/>
   <xacro:wheel prefix="back" reflect="1" rotate="2" front_set="1"/>

Commit message: Added basefootprint

File: v2mini_description/urdf/v2mini_body.urdf.xacro (robot description, xacro)
@@ -36,4 +36,9 @@
   </link>
   <link name="base_footprint"/>
+  <joint name="base_footprint_joint">
+    <origin xyz="0 0 0" rpy="0 0 0"/>
+    <parent_link="base_link"/>
+    <child_link="base_footprint"/>
+  </joint>
   <xacro:wheel prefix="front" reflect="-1" rotate="0" front_set="1"/>
   <xacro:wheel prefix="back" reflect="1" rotate="2" front_set="1"/>

File: v2mini_description/urdf/v2mini_head.urdf.xacro (robot description, xacro)
@@ -38,4 +38,5 @@
     <limit effort="1000.0" lower="0.3" upper="-0.5" velocity="0.1"/>
   </joint>
+  <!-- Attach R200 -->
 </xacro:macro>
 </robot>

File: v2mini_description/urdf/v2mini_robot.urdf.xacro (robot description, xacro)
@@ -45,4 +45,4 @@
   <xacro:arm/>
   <xacro:head/>
-  <xacro:sensor_r200 parent="head_link"/>
+  <xacro:realsense_r200 parent="head_link"/>
 </robot>

Commit message: Fixed syntax for joint

File: v2mini_description/urdf/v2mini_body.urdf.xacro (robot description, xacro)
@@ -38,6 +38,6 @@
   <joint name="base_footprint_joint">
     <origin xyz="0 0 0" rpy="0 0 0"/>
-    <parent_link="base_link"/>
-    <child_link="base_footprint"/>
+    <parent link="base_link"/>
+    <child link="base_footprint"/>
   </joint>
   <xacro:wheel prefix="front" reflect="-1" rotate="0" front_set="1"/>

Commit message: bug sim changes

File: v2mini_description/urdf/v2mini_body.urdf.xacro (robot description, xacro)
@@ -36,5 +36,5 @@
   </link>
   <link name="base_footprint"/>
-  <joint name="base_footprint_joint">
+  <joint name="base_footprint_joint" type="fixed">
     <origin xyz="0 0 0" rpy="0 0 0"/>
     <parent link="base_link"/>

Commit message: Remove collisions because of lag for now, bounding boxes later

File: v2mini_description/urdf/v2mini_body.urdf.xacro (robot description, xacro)
@@ -58,10 +58,4 @@
       </geometry>
     </visual>
-    <collision>
-       <origin xyz="0 0 0" rpy="0 0 0"/>
-       <geometry>
-           <mesh filename="package://v2mini_description/meshes/torso/torso.dae" />
-       </geometry>
-    </collision>
   </link>
   <joint name="torso_slide" type="prismatic">
@@ -87,10 +81,4 @@
        <inertia ixx="1.0" ixy="0.0" ixz="0.0" iyy="1.0" iyz="0.0" izz="1.0"/>
     </inertial>
-    <collision>
-      <origin xyz="0 0 0" rpy="0 0 0">
-      <geometry>
-        <mesh filename="package://v2mini_description/meshes/base/base_wheel.dae"/>
-      </geometry>
-    </collision>
   </link>
   <joint name="${prefix}_axel" type="continuous">

File: v2mini_description/urdf/v2mini_head.urdf.xacro (robot description, xacro)
@@ -10,10 +10,4 @@
       </geometry>
     </visual>
-      <collision>
-      <origin xyz="0 0 0" rpy="0 0 0"/>
-      <geometry>
-        <mesh filename="package://v2mini_description/meshes/head/neck.dae"/>
-      </geometry>
-      </collision>
      <inertial>
        <origin xyz="0 0 0" rpy="0 0 0"/>
@@ -29,10 +23,4 @@
        </geometry>
     </visual>
-      <collision>
-      <origin xyz="0 0 0" rpy="0 0 0"/>
-      <geometry>
-        <mesh filename="package://v2mini_description/meshes/head/head.dae"/>
-      </geometry>
-      </collision>
      <inertial>
        <origin xyz="0 0 0" rpy="0 0 0"/>
