Commit message: Added collisions and new dae

File: v2mini_description/urdf/v2mini_arm.urdf.xacro (robot description, xacro)
@@ -12,5 +12,4 @@
         <mesh filename="package://v2mini_description/meshes/arm/arm_link1.dae" />
       </geometry>
-      <material name="black"/>
     </visual>
     <collision>
@@ -33,5 +32,4 @@
         <mesh filename="package://v2mini_description/meshes/arm/arm_link2.dae" />
       </geometry>
-      <material name="grey"/>
     </visual>
     <collision>
@@ -47,5 +45,5 @@
     </inertial>
   </link>
-  <joint name="arm_joint1" type="revolute">
+  <joint name="arm_joint1" type="continuous">
     <parent link="arm_link1"/>
     <child link="arm_link2"/>
@@ -53,8 +51,8 @@
     <limit effort="1000.0" lower="-0.2" upper="2.85" velocity="0.1"/>
   </joint>
-  <xacro:arm_link num="3" mat="black" par_num="2" axis="-1 0 0" offset="0.026 0 0" j_rpy="${pi/2} 0 ${3*pi/2}" l_rpy="0 ${-pi/2}  ${-pi/2}" limit_low="-0.3" limit_high="1.6"/>
-  <xacro:arm_link num="4" mat="grey" par_num="3" axis="1 0 0" offset=" 0 0 -0.0855" j_rpy="0 ${pi/2} 0" l_rpy="${pi/2} ${pi}  0" limit_low="-3"  limit_high="3"/>
-  <xacro:arm_link num="5" mat="black" par_num="4" axis="-1 0 0" offset="0.026 0 0" j_rpy=" ${-pi/2} 0 ${pi/2}" l_rpy="${-pi/2} 0 ${-pi/2}" limit_low="-1.5" limit_high="1.5"/>
-  <xacro:arm_link num="6" mat="red" par_num="5" axis="-1 0 0" offset="0  0 -0.0415" j_rpy="${-pi/2} ${-pi/2} 0" l_rpy="${pi/2} ${pi/2} 0" limit_low="-3"  limit_high="3"/>
+  <xacro:arm_link num="3" par_num="2" axis="-1 0 0" offset="0.026 0 0" j_rpy="${pi/2} 0 ${3*pi/2}" l_rpy="0 ${-pi/2}  ${-pi/2}" limit_low="-0.3" limit_high="1.6"/>
+  <xacro:arm_link num="4" par_num="3" axis="1 0 0" offset=" 0 0 -0.0855" j_rpy="0 ${pi/2} 0" l_rpy="${pi/2} ${pi}  0" limit_low="-3"  limit_high="3"/>
+  <xacro:arm_link num="5" par_num="4" axis="-1 0 0" offset="0.026 0 0" j_rpy=" ${-pi/2} 0 ${pi/2}" l_rpy="${-pi/2} 0 ${-pi/2}" limit_low="-1.5" limit_high="1.5"/>
+  <xacro:arm_link num="6" par_num="5" axis="-1 0 0" offset="0  0 -0.0415" j_rpy="${-pi/2} ${-pi/2} 0" l_rpy="${pi/2} ${pi/2} 0" limit_low="-3"  limit_high="3"/>
   <joint name="ee_joint" type="fixed">
       <parent link="arm_link6"/>
@@ -78,5 +76,5 @@
 </xacro:macro>
 <!-- macro for the rest of the links -->
-<xacro:macro name="arm_link" params="num mat par_num axis offset j_rpy l_rpy limit_low limit_high ">
+<xacro:macro name="arm_link" params="num par_num axis offset j_rpy l_rpy limit_low limit_high ">
   <link name="arm_link${num}">
     <visual>
@@ -85,5 +83,4 @@
         <mesh filename="package://v2mini_description/meshes/arm/arm_link${num}.dae" />
       </geometry>
-      <material name="${mat}"/>
     </visual>
     <collision>
@@ -99,5 +96,5 @@
     </inertial>
   </link>
-  <joint name="arm_joint${par_num}" type="revolute">
+  <joint name="arm_joint${par_num}" type="continuous">
     <parent link="arm_link${par_num}"/>
     <child link="arm_link${num}"/>

File: v2mini_description/urdf/v2mini_body.urdf.xacro (robot description, xacro)
@@ -26,5 +26,4 @@
         <mesh filename="package://v2mini_description/meshes/base/base.dae" />
       </geometry>
-      <material name="white"/>
     </visual>
     <collision>
@@ -38,6 +37,6 @@
   <joint name="base_footprint_joint" type="fixed">
     <origin xyz="0 0 0" rpy="0 0 0"/>
-    <parent link="base_link"/>
-    <child link="base_footprint"/>
+    <parent link="base_footprint"/>
+    <child link="base_link"/>
   </joint>
   <xacro:wheel prefix="front" reflect="-1" rotate="0" front_set="1"/>
@@ -58,6 +57,11 @@
         <mesh filename="package://v2mini_description/meshes/torso/torso.dae" />
       </geometry>
-      <material name="white"/>
     </visual>
+    <collision>
+       <origin xyz="0 0 0" rpy="0 0 0"/>
+       <geometry>
+           <mesh filename="package://v2mini_description/meshes/torso/torso.dae" />
+       </geometry>
+    </collision>
   </link>
   <joint name="torso_slide" type="prismatic">
@@ -77,5 +81,4 @@
         <mesh filename="package://v2mini_description/meshes/base/base_wheel.dae" />
       </geometry>
-      <material name="red"/>
     </visual>
      <inertial>
@@ -84,4 +87,10 @@
        <inertia ixx="1.0" ixy="0.0" ixz="0.0" iyy="1.0" iyz="0.0" izz="1.0"/>
     </inertial>
+    <collision>
+      <origin xyz="0 0 0" rpy="0 0 0">
+      <geometry>
+        <mesh filename="package://v2mini_description/meshes/base/base_wheel.dae"/>
+      </geometry>
+    </collision>
   </link>
   <joint name="${prefix}_axel" type="continuous">

File: v2mini_description/urdf/v2mini_head.urdf.xacro (robot description, xacro)
@@ -9,6 +9,11 @@
         <mesh filename="package://v2mini_description/meshes/head/neck.dae" />
       </geometry>
-      <material name="black"/>
     </visual>
+      <collision>
+      <origin xyz="0 0 0" rpy="0 0 0"/>
+      <geometry>
+        <mesh filename="package://v2mini_description/meshes/head/neck.dae"/>
+      </geometry>
+      </collision>
      <inertial>
        <origin xyz="0 0 0" rpy="0 0 0"/>
@@ -22,7 +27,12 @@
       <geometry>
         <mesh filename="package://v2mini_description/meshes/head/head.dae" />
+       </geometry>
+    </visual>
+      <collision>
+      <origin xyz="0 0 0" rpy="0 0 0"/>
+      <geometry>
+        <mesh filename="package://v2mini_description/meshes/head/head.dae"/>
       </geometry>
-      <material name="yellow"/>
-    </visual>
+      </collision>
      <inertial>
        <origin xyz="0 0 0" rpy="0 0 0"/>

File: v2mini_description/urdf/v2mini_robot.urdf.xacro (robot description, xacro)
@@ -1,23 +1,4 @@
 <?xml version="1.0"?>
 <robot xmlns:xacro="http://www.ros.org/wiki/xacro" name="v2mini">
-  <!-- materials -->
-  <material name="white">
-    <color rgba="0.7 0.7 0.7 1"/>
-  </material>
-  <material name="blue">
-    <color rgba="0.3 0.3 0.9 1"/>
-  </material>
-  <material name="black">
-    <color rgba="0.2 0.2 0.2 1"/>
-  </material>
-  <material name="grey">
-    <color rgba="0.4 0.4 0.4 1"/>
-  </material>
-  <material name="yellow">
-    <color rgba="0.5 0.5 0.1 1"/>
-  </material>
-  <material name="red">
-    <color rgba="0.6 0.2 0.2 1"/>
-  </material>
   <!-- v2mini body -->
   <include filename="$(find v2mini_description)/urdf/v2mini_body.urdf.xacro" />

Commit message: positioned new robot and added new dae

File: v2mini_description/urdf/v2mini_arm.urdf.xacro (robot description, xacro)
@@ -10,13 +10,7 @@
       <origin xyz="0 0 0" rpy="0 0 0" />
       <geometry>
-        <mesh filename="package://v2mini_description/meshes/arm/arm_link1.dae" />
+        <mesh filename="package://v2mini_description/meshes/arm/arm_link1.stl" />
       </geometry>
     </visual>
-    <collision>
-      <origin xyz="0 0 0" rpy="0 0 0"/>
-      <geometry>
-         <mesh filename="package://v2mini_description/meshes/arm/arm_link1.dae" />
-      </geometry>
-    </collision>
     <inertial>
        <origin xyz="0 0 0" rpy="0 0 0"/>
@@ -30,13 +24,7 @@
       <origin xyz="0 0 0" rpy="0 ${pi} 0" />
       <geometry>
-        <mesh filename="package://v2mini_description/meshes/arm/arm_link2.dae" />
+        <mesh filename="package://v2mini_description/meshes/arm/arm_link2.stl" />
       </geometry>
     </visual>
-    <collision>
-       <origin xyz="0 0 0" rpy="0 ${pi} 0"/>
-       <geometry>
-            <mesh filename="package://v2mini_description/meshes/arm/arm_link2.dae" />
-       </geometry>
-    </collision>
    <inertial>
        <origin xyz="0 0 0" rpy="0 0 0"/>
@@ -81,13 +69,7 @@
       <origin xyz="0 0 0" rpy="${l_rpy}" />
       <geometry>
-        <mesh filename="package://v2mini_description/meshes/arm/arm_link${num}.dae" />
+        <mesh filename="package://v2mini_description/meshes/arm/arm_link${num}.stl" />
       </geometry>
     </visual>
-    <collision>
-        <origin xyz="0 0 0" rpy="${l_rpy}"/>
-        <geometry>
-            <mesh filename="package://v2mini_description/meshes/arm/arm_link${num}.dae" />
-        </geometry>
-    </collision>
     <inertial>
        <origin xyz="0 0 0" rpy="0 0 0"/>
@@ -96,5 +78,5 @@
     </inertial>
   </link>
-  <joint name="arm_joint${par_num}" type="continuous">
+  <joint name="arm_joint${par_num}" type="revolute">
     <parent link="arm_link${par_num}"/>
     <child link="arm_link${num}"/>

File: v2mini_description/urdf/v2mini_body.urdf.xacro (robot description, xacro)
@@ -10,5 +10,5 @@
 <xacro:property name="wheel_offset_radial" value="0.1405" />
 <!-- torso properties -->
-<xacro:property name="torso_offset_z" value="0.175" />
+<xacro:property name="torso_offset_z" value="0.425" />
 <xacro:property name="torso_width" value="0.2373" />
 <xacro:macro name="body">
@@ -53,5 +53,5 @@
     </inertial>
     <visual>
-      <origin xyz="0 0 0" rpy="0 0 0" />
+      <origin xyz="0 0 ${torso_offset_z}" rpy="0 0 0" />
       <geometry>
         <mesh filename="package://v2mini_description/meshes/torso/torso.dae" />
@@ -62,5 +62,5 @@
     <parent link="base_link"/>
     <child link="torso_link"/>
-    <origin xyz="0 0 ${base_offset_z}"/>
+    <origin xyz="0 0 0"/>
     <axis xyz="0 0 1"/>
     <limit effort="10" lower="-0.09" upper="0" velocity="0.5"/>

File: v2mini_description/urdf/v2mini_head.urdf.xacro (robot description, xacro)
@@ -1,9 +1,9 @@
 <?xml version="1.0"?>
 <robot xmlns:xacro="http://www.ros.org/wiki/xacro" name="v2mini">
-<xacro:property name="head_offset_z" value="0.495215" />
+<xacro:property name="head_offset_z" value="0.427" />
 <xacro:macro name="head">
   <link name="neck_link">
     <visual>
-      <origin xyz="0 0 0" rpy="0 0 0" />
+      <origin xyz="0 0 0.42" rpy="0 0 0" />
       <geometry>
         <mesh filename="package://v2mini_description/meshes/head/neck.dae" />
@@ -33,5 +33,5 @@
     <child link="head_link"/>
     <axis xyz="1 0 0"/>
-    <origin xyz="0 0 ${head_offset_z}"/>
+    <origin xyz="0 0 ${head_offset_z}" rpy="0 0 3.14"/>
     <limit effort="1000.0" lower="0.3" upper="-0.5" velocity="0.1"/>
   </joint>
