Commit message: Swapped limits, head spawns upright

File: v2mini_description/urdf/v2mini_head.urdf.xacro (robot description, xacro)
@@ -34,5 +34,5 @@
     <axis xyz="1 0 0"/>
     <origin xyz="0 0 ${head_offset_z}" rpy="0 0 3.14"/>
-    <limit effort="1000.0" lower="0.3" upper="-0.5" velocity="0.1"/>
+    <limit effort="1000.0" lower="-0.5" upper="0.3" velocity="0.1"/>
   </joint>
   <!-- Attach R200 -->
