Commit message: Update

File: v2mini_description/urdf/v2mini.urdf (robot description, URDF)
Before this commit: robot v2mini, 24 links, 23 joints
Links:
- removed link camera_ir2_frame
- removed link camera_ir2_optical_frame
- removed link camera_ir_frame
- removed link camera_ir_optical_frame
- link arm_link1: mass None -> 0.01; geometry collision mesh filename=package://v2mini_description/meshes/arm/arm_link1.dae; visual mesh filename=package://v2mini_description/meshes/arm/arm_link1.dae
- link arm_link2: mass None -> 0.01; geometry collision mesh filename=package://v2mini_description/meshes/arm/arm_link2.dae; visual mesh filename=package://v2mini_description/meshes/arm/arm_link2.dae
- link arm_link3: mass None -> 0.01; geometry collision mesh filename=package://v2mini_description/meshes/arm/arm_link3.dae; visual mesh filename=package://v2mini_description/meshes/arm/arm_link3.dae
- link arm_link4: mass None -> 0.01; geometry collision mesh filename=package://v2mini_description/meshes/arm/arm_link4.dae; visual mesh filename=package://v2mini_description/meshes/arm/arm_link4.dae
- link arm_link5: mass None -> 0.01; geometry collision mesh filename=package://v2mini_description/meshes/arm/arm_link5.dae; visual mesh filename=package://v2mini_description/meshes/arm/arm_link5.dae
- link arm_link6: mass None -> 0.01; geometry collision mesh filename=package://v2mini_description/meshes/arm/arm_link6.dae; visual mesh filename=package://v2mini_description/meshes/arm/arm_link6.dae
- link back_wheel: mass None -> 1; geometry visual mesh filename=package://v2mini_description/meshes/base/base_wheel.dae
- link base_link: mass 1 -> 10; geometry collision cylinder length=0.132 radius=0.175; visual mesh filename=package://v2mini_description/meshes/base/base.dae
- link camera_link: geometry visual box size=0.102 0.0038 0.0095
- link ee_link: mass None -> 1
- link front_wheel: mass None -> 1; geometry visual mesh filename=package://v2mini_description/meshes/base/base_wheel.dae
- link head_link: mass None -> 1; geometry visual mesh filename=package://v2mini_description/meshes/head/head.dae
- link left_wheel: mass None -> 1; geometry visual mesh filename=package://v2mini_description/meshes/base/base_wheel.dae
- link neck_link: mass None -> 1; geometry visual mesh filename=package://v2mini_description/meshes/head/neck.dae
- link right_wheel: mass None -> 1; geometry visual mesh filename=package://v2mini_description/meshes/base/base_wheel.dae
- link torso_link: mass 1 -> 5; geometry visual mesh filename=package://v2mini_description/meshes/torso/torso.dae
Joints:
- removed joint camera_ir2_joint
- removed joint camera_ir2_optical_joint
- removed joint camera_ir_joint
- removed joint camera_ir_optical_joint
- joint arm_joint1: limit lower=-3.1 upper=3.1 effort=1000.0 velocity=0.1 -> lower=-0.2 upper=2.85 effort=1000.0 velocity=0.1
- joint arm_joint2: limit lower=-1.7 upper=1.7 effort=1000.0 velocity=0.1 -> lower=-0.3 upper=1.6 effort=1000.0 velocity=0.1
- joint arm_joint3: limit lower=-3.1 upper=3.1 effort=1000.0 velocity=0.1 -> lower=-3 upper=3 effort=1000.0 velocity=0.1
- joint arm_joint4: limit lower=-3 upper=3 effort=1000.0 velocity=0.1 -> lower=-1.5 upper=1.5 effort=1000.0 velocity=0.1
- joint arm_joint5: limit lower=-3.1 upper=3.1 effort=1000.0 velocity=0.1 -> lower=-3 upper=3 effort=1000.0 velocity=0.1
- joint camera_depth_optical_joint: origin xyz=0 0 0 rpy=0 0 0 -> xyz=0 0 0 rpy=-1.570795 0 0
- joint camera_rgb_joint: origin xyz=0 0 0 rpy=0 0 0 -> xyz=0 0 0 rpy=-1.570795 0 0

File: v2mini_description/urdf/v2mini_arm.urdf.xacro (robot description, xacro)
@@ -10,5 +10,5 @@
       <origin xyz="0 0 0" rpy="0 0 0" />
       <geometry>
-        <mesh filename="package://v2mini_description/meshes/arm/arm_link1.stl" />
+        <mesh filename="package://v2mini_description/meshes/arm/arm_link1.dae" />
       </geometry>
       <material name="black"/>
@@ -17,5 +17,5 @@
       <origin xyz="0 0 0" rpy="0 0 0"/>
       <geometry>
-         <mesh filename="package://v2mini_description/meshes/arm/arm_link1.stl" />
+         <mesh filename="package://v2mini_description/meshes/arm/arm_link1.dae" />
       </geometry>
     </collision>
@@ -31,5 +31,5 @@
       <origin xyz="0 0 0" rpy="0 ${pi} 0" />
       <geometry>
-        <mesh filename="package://v2mini_description/meshes/arm/arm_link2.stl" />
+        <mesh filename="package://v2mini_description/meshes/arm/arm_link2.dae" />
       </geometry>
       <material name="grey"/>
@@ -38,5 +38,5 @@
        <origin xyz="0 0 0" rpy="0 ${pi} 0"/>
        <geometry>
-            <mesh filename="package://v2mini_description/meshes/arm/arm_link2.stl" />
+            <mesh filename="package://v2mini_description/meshes/arm/arm_link2.dae" />
        </geometry>
     </collision>
@@ -83,5 +83,5 @@
       <origin xyz="0 0 0" rpy="${l_rpy}" />
       <geometry>
-        <mesh filename="package://v2mini_description/meshes/arm/arm_link${num}.stl" />
+        <mesh filename="package://v2mini_description/meshes/arm/arm_link${num}.dae" />
       </geometry>
       <material name="${mat}"/>
@@ -90,5 +90,5 @@
         <origin xyz="0 0 0" rpy="${l_rpy}"/>
         <geometry>
-            <mesh filename="package://v2mini_description/meshes/arm/arm_link${num}.stl" />
+            <mesh filename="package://v2mini_description/meshes/arm/arm_link${num}.dae" />
         </geometry>
     </collision>

File: v2mini_description/urdf/v2mini_body.urdf.xacro (robot description, xacro)
@@ -24,5 +24,5 @@
       <origin xyz="0 0 ${base_offset_z}" rpy="0 0 0" />
       <geometry>
-        <mesh filename="package://v2mini_description/meshes/base/base.stl" />
+        <mesh filename="package://v2mini_description/meshes/base/base.dae" />
       </geometry>
       <material name="white"/>
@@ -50,5 +50,5 @@
       <origin xyz="0 0 0" rpy="0 0 0" />
       <geometry>
-        <mesh filename="package://v2mini_description/meshes/torso/torso.stl" />
+        <mesh filename="package://v2mini_description/meshes/torso/torso.dae" />
       </geometry>
       <material name="white"/>
@@ -69,5 +69,5 @@
       <origin xyz="0 0 0" rpy="0 0 ${pi/2*rotate}"/>
       <geometry>
-        <mesh filename="package://v2mini_description/meshes/base/base_wheel.stl" />
+        <mesh filename="package://v2mini_description/meshes/base/base_wheel.dae" />
       </geometry>
       <material name="red"/>

File: v2mini_description/urdf/v2mini_head.urdf.xacro (robot description, xacro)
@@ -7,5 +7,5 @@
       <origin xyz="0 0 0" rpy="0 0 0" />
       <geometry>
-        <mesh filename="package://v2mini_description/meshes/head/neck.stl" />
+        <mesh filename="package://v2mini_description/meshes/head/neck.dae" />
       </geometry>
       <material name="black"/>
@@ -21,5 +21,5 @@
       <origin xyz="0 0 0" rpy="0 0 0" />
       <geometry>
-        <mesh filename="package://v2mini_description/meshes/head/head.stl" />
+        <mesh filename="package://v2mini_description/meshes/head/head.dae" />
       </geometry>
       <material name="yellow"/>

Commit message: Added dae so it can work in gzweb

File: v2mini_description/urdf/v2mini.urdf (robot description, URDF)
Before this commit: robot v2mini, 20 links, 19 joints
Links:
- removed link camera_depth_frame
- removed link camera_depth_optical_frame
- removed link camera_link
- removed link camera_rgb_frame
- removed link camera_rgb_optical_frame
- added link base_footprint
- link arm_link1: geometry visual mesh filename=package://v2mini_description/meshes/arm/arm_link1.stl
- link arm_link2: geometry visual mesh filename=package://v2mini_description/meshes/arm/arm_link2.stl
- link arm_link3: geometry visual mesh filename=package://v2mini_description/meshes/arm/arm_link3.stl
- link arm_link4: geometry visual mesh filename=package://v2mini_description/meshes/arm/arm_link4.stl
- link arm_link5: geometry visual mesh filename=package://v2mini_description/meshes/arm/arm_link5.stl
- link arm_link6: geometry visual mesh filename=package://v2mini_description/meshes/arm/arm_link6.stl
Joints:
- removed joint camera_depth_joint
- removed joint camera_depth_optical_joint
- removed joint camera_joint
- removed joint camera_rgb_joint
- removed joint camera_rgb_optical_joint
- added joint base_footprint_joint: type fixed, parent base_footprint, child base_link, origin xyz=0 0 0 rpy=0 0 0
- joint arm_joint1: type revolute -> continuous
- joint neck_tilt: limit lower=0.3 upper=-0.5 effort=1000.0 velocity=0.1 -> lower=-0.5 upper=0.3 effort=1000.0 velocity=0.1; origin xyz=0 0 0.495215 -> xyz=0 0 0.427 rpy=0 0 3.14
- joint torso_slide: origin xyz=0 0 0.0192 -> xyz=0 0 0

File: v2mini_description/urdf/v2mini_head.urdf.xacro (robot description, xacro)
@@ -28,4 +28,10 @@
        <inertia ixx="1.0" ixy="0.0" ixz="0.0" iyy="1.0" iyz="0.0" izz="1.0"/>
     </inertial>
+    <collision>
+     <origin xyz="0 0 0" rpy="0 0 0"/>
+     <geometry>
+        <box size="0 0 0"/>
+     </geometry>
+    </collision>
   </link>
   <joint name="neck_tilt" type="revolute">

File: v2mini_description/urdf/v2mini_robot.urdf.xacro (robot description, xacro)
@@ -21,5 +21,5 @@
     <parent link="torso_link"/>
     <child link="arm_link1"/>
-    <origin xyz="0 0 0"/>
+    <origin xyz="0 0 0" rpy="0 0 0"/>
   </joint>
   <xacro:body/>
