Commit message: remove web stuff

File: v2mini_description/urdf/sensors/r200.urdf.xacro (robot description, xacro)
@@ -47,5 +47,5 @@
        <origin xyz="${-r200_cam_rgb_px + -r200_cam_px} ${-r200_cam_rgb_py + -r200_cam_py} ${-r200_cam_rgb_pz + -r200_cam_pz}" rpy="${M_PI/2} 0 ${M_PI/2}"/>
         <geometry>
-         <mesh filename="package://realsense_r200_description/meshes/realsense_r200.dae"/>
+         <mesh filename="package://v2mini_description/meshes/sensors/realsense_r200.dae"/>
         </geometry>
       </visual>

Commit message: Change filepath name for r200 dae

File: v2mini_description/urdf/sensors/r200.urdf.xacro (robot description, xacro)
@@ -47,5 +47,5 @@
        <origin xyz="${-r200_cam_rgb_px + -r200_cam_px} ${-r200_cam_rgb_py + -r200_cam_py} ${-r200_cam_rgb_pz + -r200_cam_pz}" rpy="${M_PI/2} 0 ${M_PI/2}"/>
         <geometry>
-         <mesh filename="package://v2mini_description/meshes/sensors/realsense_r200.dae"/>
+         <mesh filename="package://v2mini_description/meshes/sensors/r200.dae"/>
         </geometry>
       </visual>
